Commit message: fix(sim): fixes inertia of wheels

File: src/wallington_description/urdf/wallington.urdf.xacro (robot description, xacro)
@@ -34,5 +34,5 @@
     <link name="front_left_wheel_link">
         <inertial>
-            <origin xyz="0 0 0.025" rpy="0 0 0"/>
+            <origin xyz="0 0 0" rpy="0 0 0"/>
             <mass value="0.1"/>
             <inertia ixx="1.645833e-5" ixy="0.0" ixz="0.0"
@@ -62,5 +62,5 @@
     <link name="front_right_wheel_link">
         <inertial>
-            <origin xyz="0 0 0.025" rpy="0 0 0"/>
+            <origin xyz="0 0 0" rpy="0 0 0"/>
             <mass value="0.1"/>
             <inertia ixx="1.645833e-5" ixy="0.0" ixz="0.0"
@@ -90,5 +90,5 @@
     <link name="back_left_wheel_link">
         <inertial>
-            <origin xyz="0 0 0.025" rpy="0 0 0"/>
+            <origin xyz="0 0 0" rpy="0 0 0"/>
             <mass value="0.1"/>
             <inertia ixx="1.645833e-5" ixy="0.0" ixz="0.0"
@@ -118,5 +118,5 @@
     <link name="back_right_wheel_link">
         <inertial>
-            <origin xyz="0 0 0.025" rpy="0 0 0"/>
+            <origin xyz="0 0 0" rpy="0 0 0"/>
             <mass value="0.1"/>
             <inertia ixx="1.645833e-5" ixy="0.0" ixz="0.0"
